File: Hardware/PCB/CAD/xmasOrnament2024.kicad_sch (KiCad schematic)
At the start: 56 parts, among them IC1 TP4056-42, Q1 AO3401A, Q2 CJ3400, SW1 BZCN_TSA007A1518B03, SW2 BZCN_TSA007A1518B03, U1 STM32C011F6, U2 TPS7A2633DRVR

Commit message: Updated buzzer component values.
Parts:
- C7: value 10n -> 2u2
- R10: value 22R -> 100R
Changed lines of the file:
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@@
 (kicad_sch
-	(version 20231120)
+	(version 20250114)
 	(generator "eeschema")
-	(generator_version "8.0")
+	(generator_version "9.0")
 	(paper "A4")
+	(rectangle
+		(start 101.6 97.79)
+		(end 123.19 118.11)
+		(stroke
+			(width 0)
+			(type dot)
+		)
+		(fill
+			(type none)
+		)
+	)
+	(rectangle
+		(start 129.54 82.55)
+		(end 278.13 132.08)
+		(stroke
+			(width 0)
+			(type dash)
+		)
+		(fill
+			(type none)
+		)
+	)
+	(rectangle
+		(start 13.97 82.55)
+		(end 127 132.08)
+		(stroke
+			(width 0)
+			(type dash)
+		)
+		(fill
+			(type none)
+		)
+	)
+	(rectangle
+		(start 13.97 13.97)
+		(end 127 80.01)
+		(stroke
+			(width 0)
+			(type dash)
+		)
+		(fill
+			(type none)
+		)
+	)
+	(rectangle
+		(start 129.54 13.97)
+		(end 278.13 80.01)
+		(stroke
+			(width 0)
+			(type dash)
+		)
+		(fill
+			(type none)
+		)
+	)
+	(text "INPUT & OUTPUT PERIPHERAL"
+		(exclude_from_sim no)
+		(at 145.034 16.256 0)
+		(effects
+			(font
+				(size 1.27 1.27)
+			)
+		)
+	)
+	(text "POWER & CHARGER"
+		(exclude_from_sim no)
+		(at 24.13 16.002 0)
+		(effects
+			(font
+				(size 1.27 1.27)
+			)
+		)
+	)
+	(text "WS ADDRESSABLE LEDS"
+		(exclude_from_sim no)
+		(at 141.986 85.09 0)
+		(effects
+			(font
+				(size 1.27 1.27)
+			)
+		)
+	)
+	(text "MCU PROGRAMMING"
+		(exclude_from_sim no)
+		(at 101.6 97.79 0)
+		(effects
+			(font
+				(size 1.27 1.27)
+			)
+			(justify left bottom)
+		)
+	)
 	(junction
 		(at 31.75 57.15)
@@
 		)
 	)
-	(rectangle
-		(start 101.6 97.79)
-		(end 123.19 118.11)
-		(stroke
-			(width 0)
-			(type dot)
-		)
-		(fill
-			(type none)
-		)
-	)
-	(rectangle
-		(start 129.54 82.55)
-		(end 278.13 132.08)
-		(stroke
-			(width 0)
-			(type dash)
-		)
-		(fill
-			(type none)
-		)
-	)
-	(rectangle
-		(start 13.97 82.55)
-		(end 127 132.08)
-		(stroke
-			(width 0)
-			(type dash)
-		)
-		(fill
-			(type none)
-		)
-	)
-	(rectangle
-		(start 13.97 13.97)
-		(end 127 80.01)
-		(stroke
-			(width 0)
-			(type dash)
-		)
-		(fill
-			(type none)
-		)
-	)
-	(rectangle
-		(start 129.54 13.97)
-		(end 278.13 80.01)
-		(stroke
-			(width 0)
-			(type dash)
-		)
-		(fill
-			(type none)
-		)
-	)
-	(text "INPUT & OUTPUT PERIPHERAL"
-		(exclude_from_sim no)
-		(at 145.034 16.256 0)
-		(effects
-			(font
-				(size 1.27 1.27)
-			)
-		)
-	)
-	(text "POWER & CHARGER"
-		(exclude_from_sim no)
-		(at 24.13 16.002 0)
-		(effects
-			(font
-				(size 1.27 1.27)
-			)
-		)
-	)
-	(text "WS ADDRESSABLE LEDS"
-		(exclude_from_sim no)
-		(at 141.986 85.09 0)
-		(effects
-			(font
-				(size 1.27 1.27)
-			)
-		)
-	)
-	(text "MCU PROGRAMMING"
-		(exclude_from_sim no)
-		(at 101.6 97.79 0)
-		(effects
-			(font
-				(size 1.27 1.27)
-			)
-			(justify left bottom)
-		)
-	)
 	(label "BTN1"
 		(at 184.15 38.1 180)
-		(fields_autoplaced yes)
 		(effects
 			(font
@@
 	(label "BUZZER"
 		(at 91.44 123.19 180)
-		(fields_autoplaced yes)
 		(effects
 			(font
@@
 	(label "RST"
 		(at 121.92 115.57 180)
-		(fields_autoplaced yes)
 		(effects
 			(font
@@
 	(label "RST"
 		(at 45.72 102.87 0)
-		(fields_autoplaced yes)
 		(effects
 			(font
@@
 	(label "SW_CLK"
 		(at 105.41 90.17 180)
-		(fields_autoplaced yes)
 		(effects
 			(font
@@
 	(label "GND"
 		(at 121.92 100.33 180)
-		(fields_autoplaced yes)
 		(effects
 			(font
@@
 	(label "RST"
 		(at 80.01 90.17 180)
-		(fields_autoplaced yes)
 		(effects
 			(font
@@
 	(label "BTN2"
 		(at 45.72 115.57 0)
-		(fields_autoplaced yes)
 		(effects
 			(font
@@
 	(label "PERIPH_SUPPLY"
 		(at 91.44 115.57 180)
-		(fields_autoplaced yes)
 		(effects
 			(font
@@
 	(label "BTN1"
 		(at 45.72 120.65 0)
-		(fields_autoplaced yes)
 		(effects
 			(font
@@
 	(label "SW_CLK"
 		(at 121.92 107.95 180)
-		(fields_autoplaced yes)
 		(effects
 			(font
@@
 	(label "BTN2"
 		(at 184.15 57.15 180)
-		(fields_autoplaced yes)
 		(effects
 			(font
@@
 	(label "PERIPH_SUPPLY"
 		(at 54.61 67.31 0)
-		(fields_autoplaced yes)
 		(effects
 			(font
@@
 	(label "SW_CLK"
 		(at 91.44 102.87 180)
-		(fields_autoplaced yes)
 		(effects
 			(font
@@
 	(label "WS_DIN"
 		(at 91.44 118.11 180)
-		(fields_autoplaced yes)
 		(effects
 			(font
@@
 	(label "3V3"
 		(at 121.92 104.14 180)
-		(fields_autoplaced yes)
 		(effects
 			(font
@@
 	(label "WS_DIN"
 		(at 130.81 99.06 0)
-		(fields_autoplaced yes)
 		(effects
 			(font
@@
 	(label "SW_DIO"
 		(at 91.44 105.41 180)
-		(fields_autoplaced yes)
 		(effects
 			(font
@@
 	(label "SW_DIO"
 		(at 121.92 111.76 180)
-		(fields_autoplaced yes)
 		(effects
 			(font
@@
 	(label "BUZZER"
 		(at 196.85 52.07 0)
-		(fields_autoplaced yes)
 		(effects
 			(font
@@
 			)
 		)
-		(property "Value" "22R"
+		(property "Value" "100R"
 			(at 236.728 31.242 0)
 			(effects
@@
 			)
 		)
-		(property "Value" "10n"
+		(property "Value" "2u2"
 			(at 231.902 40.64 0)
 			(effects
@@
 		)
 	)
+	(embedded_fonts no)
 )
